Commit message: husky + ur5e combined - still they are intersecting (will be fixed later) - mobile base movement is unstable NEXT STEPS: -  publish a task topic with a converted coord. and rviz subscribes it to show the point in rviz2 - (additionally) rviz piont cloud are too blunt - gazebo receives a transformation matrix and reposition the ifc world model to be aligned with the point cloud model
Co-authored-by: Copilot <copilot@github.com>

File: src/robot_gazebo/models/robots/husky/husky.urdf (robot description, URDF)
Before this commit: robot husky_robot, 11 links, 10 joints
Links:
- removed link imu_link
- link base_link: geometry collision box size=1.0074 0.5709 0.2675; visual mesh filename=model://husky/meshes/base_link.stl scale=1 1 1
- link front_bumper_link: geometry visual mesh filename=model://husky/meshes/bumper.stl scale=1 1 1
- link front_left_wheel_link: geometry collision cylinder length=0.1143 radius=0.17775; visual mesh filename=model://husky/meshes/wheel.stl scale=1 1 1
- link front_right_wheel_link: geometry collision cylinder length=0.1143 radius=0.17775; visual mesh filename=model://husky/meshes/wheel.stl scale=1 1 1
- link rear_bumper_link: geometry visual mesh filename=model://husky/meshes/bumper.stl scale=1 1 1
- link rear_left_wheel_link: geometry collision cylinder length=0.1143 radius=0.17775; visual mesh filename=model://husky/meshes/wheel.stl scale=1 1 1
- link rear_right_wheel_link: geometry collision cylinder length=0.1143 radius=0.17775; visual mesh filename=model://husky/meshes/wheel.stl scale=1 1 1
- link top_plate_link: geometry visual mesh filename=model://husky/meshes/top_plate.stl scale=1 1 1
- link user_rail_link: geometry visual mesh filename=model://husky/meshes/user_rail.stl scale=1 1 1
Joints:
- removed joint imu_joint
