Commit message: task / matrix topic publisher added
Co-authored-by: Copilot <copilot@github.com>

File: src/robot_gazebo/models/robots/husky5e/husky5e.urdf (robot description, URDF)
Before this commit: robot husky5e, 23 links, 22 joints
Links:
- removed link robot_plate_link
- added link ur_plate_link, mass 1.0; collision box size=0.55 0.40 0.01; visual box size=0.55 0.40 0.01
Joints:
- removed joint robot_plate_joint
- added joint ur_plate_joint: type fixed, parent base_link, child ur_plate_link, origin xyz=0 0 0.245 rpy=0 0 0
- joint arm_mount_joint: parent robot_plate_link -> ur_plate_link
