Commit message: code cleaned && husky setup for creating a husky + ur5e wrapper done

File: src/robot_gazebo/models/robots/husky5e.urdf (robot description, URDF)
Before this commit: robot husky5e, 23 links, 22 joints
Links:
- removed link ur_plate_link
- added link robot_plate_link, mass 1.0; collision box size=0.55 0.40 0.01; visual box size=0.55 0.40 0.01
Joints:
- removed joint ur_plate_joint
- added joint robot_plate_joint: type fixed, parent base_link, child robot_plate_link, origin xyz=0 0 0.245 rpy=0 0 0
- joint arm_mount_joint: parent ur_plate_link -> robot_plate_link

File: src/robot_gazebo/urdf/ur5e/ur5e.xacro (robot description, xacro)
@@ -14,5 +14,5 @@
     Refer to 'inc/ur_macro.xacro' for more information.
   -->
-  <xacro:include filename="$(find ur_description)/urdf/inc/ur5e_macro.xacro"/>
+  <xacro:include filename="$(find robot_gazebo)/urdf/ur5e/inc/ur5e_macro.xacro"/>
   <xacro:ur5e_robot prefix="" />
 </robot>
