Commit message: robot spawning & removing fixed

File: src/robot_gazebo/models/robots/husky_ur5e.urdf (robot description, URDF)
Before this commit: robot husky_ur5e, 24 links, 23 joints
Links:
- link base_link: geometry collision box size=0.7899200000000001 0.5709 0.10375; collision box size=0.9874 0.5709 0.12375
- link front_left_wheel: geometry collision cylinder length=0.1143 radius=0.1651; collision mesh filename=model://a200_meshes/collision/wheel.stl
- link front_right_wheel: geometry collision cylinder length=0.1143 radius=0.1651; collision mesh filename=model://a200_meshes/collision/wheel.stl
- link rear_left_wheel: geometry collision cylinder length=0.1143 radius=0.1651; collision mesh filename=model://a200_meshes/collision/wheel.stl
- link rear_right_wheel: geometry collision cylinder length=0.1143 radius=0.1651; collision mesh filename=model://a200_meshes/collision/wheel.stl
- link top_chassis_link: geometry collision mesh filename=model://a200_meshes/collision/top_chassis.stl; visual mesh filename=model://a200_meshes/visual/top_chassis.dae
- link ur_arm_base_link_inertia: geometry collision mesh filename=model://ur5e_meshes/collision/base.stl; visual mesh filename=model://ur5e_meshes/visual/base.dae
- link ur_arm_forearm_link: geometry collision mesh filename=model://ur5e_meshes/collision/forearm.stl; visual mesh filename=model://ur5e_meshes/visual/forearm.dae
- link ur_arm_shoulder_link: geometry collision mesh filename=model://ur5e_meshes/collision/shoulder.stl; visual mesh filename=model://ur5e_meshes/visual/shoulder.dae
- link ur_arm_upper_arm_link: geometry collision mesh filename=model://ur5e_meshes/collision/upperarm.stl; visual mesh filename=model://ur5e_meshes/visual/upperarm.dae
- link ur_arm_wrist_1_link: geometry collision mesh filename=model://ur5e_meshes/collision/wrist1.stl; visual mesh filename=model://ur5e_meshes/visual/wrist1.dae
- link ur_arm_wrist_2_link: geometry collision mesh filename=model://ur5e_meshes/collision/wrist2.stl; visual mesh filename=model://ur5e_meshes/visual/wrist2.dae
- link ur_arm_wrist_3_link: geometry collision mesh filename=model://ur5e_meshes/collision/wrist3.stl; visual mesh filename=model://ur5e_meshes/visual/wrist3.dae

Commit message: moveit for motion planning wired

File: src/robot_gazebo/models/robots/husky_ur5e.urdf (robot description, URDF)
Before this commit: robot husky_ur5e, 24 links, 23 joints
Links:
- link base_link: geometry collision box size=0.7899200000000001 0.5709 0.10375; collision box size=0.9874 0.5709 0.12375
- link front_left_wheel: geometry collision cylinder length=0.1143 radius=0.1651; collision mesh filename=package://robot_gazebo/models/robots/a200_meshes/collision/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
- link front_right_wheel: geometry collision cylinder length=0.1143 radius=0.1651; collision mesh filename=package://robot_gazebo/models/robots/a200_meshes/collision/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
- link rear_left_wheel: geometry collision cylinder length=0.1143 radius=0.1651; collision mesh filename=package://robot_gazebo/models/robots/a200_meshes/collision/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
- link rear_right_wheel: geometry collision cylinder length=0.1143 radius=0.1651; collision mesh filename=package://robot_gazebo/models/robots/a200_meshes/collision/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
- link top_chassis_link: geometry collision mesh filename=package://robot_gazebo/models/robots/a200_meshes/collision/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; visual mesh filename=package://robot_gazebo/models/robots/a200_meshes/visual/top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
- link ur_arm_base_link_inertia: geometry collision mesh filename=package://robot_gazebo/models/robots/ur5e_meshes/collision/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; visual mesh filename=package://robot_gazebo/models/robots/ur5e_meshes/visual/bas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
- link ur_arm_forearm_link: geometry collision mesh filename=package://robot_gazebo/models/robots/ur5e_meshes/collision/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; visual mesh filename=package://robot_gazebo/models/robots/ur5e_meshes/visual/for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
- link ur_arm_shoulder_link: geometry collision mesh filename=package://robot_gazebo/models/robots/ur5e_meshes/collision/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; visual mesh filename=package://robot_gazebo/models/robots/ur5e_meshes/visual/sho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
- link ur_arm_upper_arm_link: geometry collision mesh filename=package://robot_gazebo/models/robots/ur5e_meshes/collision/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; visual mesh filename=package://robot_gazebo/models/robots/ur5e_meshes/visual/upp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
- link ur_arm_wrist_1_link: geometry collision mesh filename=package://robot_gazebo/models/robots/ur5e_meshes/collision/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; visual mesh filename=package://robot_gazebo/models/robots/ur5e_meshes/visual/wri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
- link ur_arm_wrist_2_link: geometry collision mesh filename=package://robot_gazebo/models/robots/ur5e_meshes/collision/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; visual mesh filename=package://robot_gazebo/models/robots/ur5e_meshes/visual/wri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
- link ur_arm_wrist_3_link: geometry collision mesh filename=package://robot_gazebo/models/robots/ur5e_meshes/collision/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; visual mesh filename=package://robot_gazebo/models/robots/ur5e_meshes/visual/wri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
