Commit message: robot stabilized && motion planning ready - thank you panos 2cm deviation from the floor & wheels with friction solved the problem - fake drill (cone) attached - rviz + gazebo synchronized

File: src/husky_ur5e_moveit_config/config/husky_ur5e.ros2_control.xacro (robot description, xacro)
@@ -5,9 +5,5 @@
         <ros2_control name="${name}" type="system">
             <hardware>
-                <!-- Mock hardware: echoes commands as state. controller_manager
-                     runs as a standalone ros2_control_node (see robot_gazebo
-                     launch). Arm motion shows in RViz only; Gazebo is the
-                     static scene + spawned base. -->
-                <plugin>mock_components/GenericSystem</plugin>
+                <plugin>gazebo_ros2_control/GazeboSystem</plugin>
             </hardware>
             <joint name="ur_arm_shoulder_pan_joint">
@@ -53,4 +49,24 @@
                 <state_interface name="velocity"/>
             </joint>
+            <joint name="front_left_wheel_joint">
+                <command_interface name="effort"/>
+                <state_interface name="position"/>
+                <state_interface name="velocity"/>
+            </joint>
+            <joint name="front_right_wheel_joint">
+                <command_interface name="effort"/>
+                <state_interface name="position"/>
+                <state_interface name="velocity"/>
+            </joint>
+            <joint name="rear_left_wheel_joint">
+                <command_interface name="effort"/>
+                <state_interface name="position"/>
+                <state_interface name="velocity"/>
+            </joint>
+            <joint name="rear_right_wheel_joint">
+                <command_interface name="effort"/>
+                <state_interface name="position"/>
+                <state_interface name="velocity"/>
+            </joint>
         </ros2_control>
     </xacro:macro>

File: src/husky_ur5e_moveit_config/config/husky_ur5e.urdf.xacro (robot description, xacro)
@@ -2,8 +2,13 @@
 <robot xmlns:xacro="http://www.ros.org/wiki/xacro" name="husky_ur5e">
     <xacro:arg name="initial_positions_file" default="initial_positions.yaml" />
-    <!-- Import husky_ur5e urdf file -->
     <xacro:include filename="$(find robot_gazebo)/models/robots/husky_ur5e.urdf" />
-    <!-- Import control_xacro -->
     <xacro:include filename="husky_ur5e.ros2_control.xacro" />
     <xacro:husky_ur5e_ros2_control name="UR5eArm" initial_positions_file="$(arg initial_positions_file)"/>
+    <gazebo>
+        <plugin name="gazebo_ros2_control" filename="libgazebo_ros2_control.so">
+            <robot_param>robot_description</robot_param>
+            <robot_param_node>robot_state_publisher</robot_param_node>
+            <parameters>$(find husky_ur5e_moveit_config)/config/ros2_controllers.yaml</parameters>
+        </plugin>
+    </gazebo>
 </robot>

File: src/robot_gazebo/models/robots/husky_ur5e.urdf (robot description, URDF)
Before this commit: robot husky_ur5e, 24 links, 23 joints
Links:
- added link drill_link, mass 0.05; collision cylinder length=0.150 radius=0.010; visual cylinder length=0.120 radius=0.010
- added link drill_tip
Joints:
- added joint drill_to_tip: type fixed, parent drill_link, child drill_tip, origin xyz=0 0 0.150 rpy=0 0 0
- added joint tool0_to_drill: type fixed, parent ur_arm_tool0, child drill_link, origin xyz=0 0 0 rpy=0 0 0
